Commit message: измененный FOV и машинка на парковке

File: robot_description/urdf/depth.urdf.xacro (robot description, xacro)
@@ -12,12 +12,12 @@
     <link name="depth_frame">
         <visual>
-            <origin xyz="0.00465 0 0" rpy="${M_PI/2} 0 ${M_PI/2}"/>
+            <origin xyz="0 0 0" rpy="${M_PI/2} 0 ${M_PI/2}"/>
             <geometry>
-                <mesh filename="file://$(find robot_description)/urdf/d455.stl" scale="0.001 0.001 0.001"/>
+                <mesh filename="file://$(find robot_description)/urdf/d455_sim.stl" scale="0.001 0.001 0.001"/>
             </geometry>
             <material name="aluminum"/>
         </visual>
         <collision>
-            <origin xyz="0.00465 0 0" rpy="${M_PI/2} 0 ${M_PI/2}"/>
+            <origin xyz="0 0 0" rpy="${M_PI/2} 0 ${M_PI/2}"/>
             <geometry>
                 <box size="0.026 0.124 0.029"/>
@@ -49,17 +49,8 @@
                     <far>10</far>
                 </clip>
-                <lens>
-                    <intrinsics>
-                    <fx>421.61578369140625</fx>
-                    <fy>421.61578369140625</fy>
-                    <cx>422.2854309082031</cx>
-                    <cy>236.57237243652344</cy>
-                    <s>0</s>
-                    </intrinsics>
-                </lens>
                 <noise>
                     <type>gaussian</type>
                     <mean>0.0</mean>
-                    <stddev>0.007</stddev>
+                    <stddev>0.003</stddev>
                 </noise>
             </camera>
@@ -71,5 +62,5 @@
             <always_on>false</always_on>
             <camera>
-                <horizontal_fov>1.20427718</horizontal_fov>
+                <horizontal_fov>1.51843645</horizontal_fov>
                 <image>
                     <width>848</width>
@@ -83,5 +74,5 @@
                     <type>gaussian</type>
                     <mean>0.0</mean>
-                    <stddev>0.007</stddev>
+                    <stddev>0.003</stddev>
                 </noise>
             </camera>

File: robot_description/urdf/lidar.urdf.xacro (robot description, xacro)
@@ -10,5 +10,5 @@
         <visual>
             <geometry>
-                <mesh filename="file://$(find robot_description)/urdf/lidar.stl" scale="0.001 0.001 0.001"/>
+                <mesh filename="file://$(find robot_description)/urdf/lidar_sim.stl" scale="0.001 0.001 0.001"/>
             </geometry>
             <material name="aluminum"/>

File: robot_description/urdf/robot.urdf.xacro (robot description, xacro)
@@ -55,5 +55,5 @@
         <visual>
             <geometry>
-                <mesh filename="file://$(find robot_description)/urdf/body_center.stl" scale="0.001 0.001 0.001"/>
+                <mesh filename="file://$(find robot_description)/urdf/body_center_sim.stl" scale="0.001 0.001 0.001"/>
             </geometry>
             <material name="blue"/>
@@ -77,5 +77,5 @@
         <visual>
             <geometry>
-                <mesh filename="file://$(find robot_description)/urdf/left_tire.stl" scale="0.001 0.001 0.001"/>
+                <mesh filename="file://$(find robot_description)/urdf/left_tire_sim.stl" scale="0.001 0.001 0.001"/>
             </geometry>
             <material name="blue"/>
@@ -106,5 +106,5 @@
         <visual>
             <geometry>
-                <mesh filename="file://$(find robot_description)/urdf/right_tire.stl" scale="0.001 0.001 0.001"/>
+                <mesh filename="file://$(find robot_description)/urdf/right_tire_sim.stl" scale="0.001 0.001 0.001"/>
             </geometry>
             <material name="blue"/>
@@ -134,5 +134,5 @@
         <visual>
             <geometry>
-                <mesh filename="file://$(find robot_description)/urdf/left_tire.stl" scale="0.0009 0.0009 0.0009"/>
+                <mesh filename="file://$(find robot_description)/urdf/left_tire_sim.stl" scale="0.0009 0.0009 0.0009"/>
             </geometry>
             <material name="white"/>
